File: electric/AFM_QFM_input.brd (EAGLE design)
At the start: 64.4 x 55.9 mm, 42 parts, among them U1 LTC3260EMSE#PBF, U2 AD5696RARUZ-RL7RU_16_ADI-M, U3 LM324KAD

Commit message: allboards
Parts:
- removed J2: (no value), SparkFun-Connectors:1X04_LONGPADS
- removed R1: 220, SparkFun-Resistors:0603
- removed R11, R12, R13: 5k, 52101-101-REV-A_v16:RC-MASTER-SMD_R0603MP
- removed R14, R15, R20: 10k, 52101-101-REV-A_v16:RC-MASTER-SMD_R0603MP
- removed R16, R17, R18, R19: 30k, 52101-101-REV-A_v16:RC-MASTER-SMD_R0603MP
- removed R2: 100k, SparkFun-Resistors:0603
- removed U$1, U$3, U$5, U$7: 2.2uf, Nordic_nRF:RESC0603_M
- removed U$2, U$4, U$6, U$8: 1uF, Nordic_nRF:RESC0603_M
- removed U$9: 4.7uf, Nordic_nRF:RESC0603_M
- added C11, C13, C15, C17: 0.1uF, SparkFun-Capacitors:0603
- added C12, C14, C16, C18, C8: 10uF, SparkFun-Capacitors:0805
- added IC1: 74HC86_SOIC, IC_Logic:SOIC127P600X175-14N
- added QFM_SENSOR: (no value), SparkFun-Connectors:1X05_LONGPADS
- added Y1: OSCILLATORSMD-5X3, SparkFun-Clocks:OSCILLATOR-SMD-5X3.2
- C1: value 1.0uF -> 0.1uF; device SparkFun-Capacitors:0805 -> SparkFun-Capacitors:0603
- C2: value 10uF -> 10nF; device SparkFun-Capacitors:0805 -> SparkFun-Capacitors:0603
- C3: value 10nF -> 0.1uF
- C4: value 10uF -> 0.1uF; device SparkFun-Capacitors:0805 -> SparkFun-Capacitors:0603
- C5: value 10nF -> 10uF; device SparkFun-Capacitors:0603 -> SparkFun-Capacitors:0805
- C6, C7: value 10uF -> 1.5nF; device SparkFun-Capacitors:0805 -> resistor:C0603
- R10: value 5k -> 3224W-1-102E; device 52101-101-REV-A_v16:RC-MASTER-SMD_R0603MP -> 3224W-1-102E:TRIM_3224W-1-102E
- R3: value 100k -> (none); device SparkFun-Resistors:0603 -> rcl:R0603
- R4, R5: value 300k -> (none); device SparkFun-Resistors:0603 -> rcl:R0603
- R6, R7, R8, R9: value 5k -> (none); device 52101-101-REV-A_v16:RC-MASTER-SMD_R0603MP -> rcl:R0603
- U1: value LTC3260EMSE#PBF -> AD9833BRM; device LTC3260EMSE_PBF (1):MSOP-16_MSE -> AD9833BRM:SOP50P490X110-10N
- U2: value AD5696RARUZ-RL7RU_16_ADI-M -> LM339D; device AD5696:RU_16_ADI-M -> LM339D:SOIC127P600X175-14N
- moved C4 51.4 mm to (6.35, 8.89), turned to 180 degrees
- moved C5 47.9 mm to (6.35, 11.4), turned to 180 degrees
- moved C1 40.5 mm to (10.2, 16.5)
- moved C6 38.2 mm to (22.9, 19.1), turned to 0 degrees
- moved U2 35.3 mm to (31.8, 45.7), turned to 90 degrees
- moved C3 33.6 mm to (10.2, 14.0), turned to 0 degrees
- moved U1 33.1 mm to (16.5, 16.5), turned to 0 degrees
- moved C2 32.5 mm to (14.0, 20.3), turned to 0 degrees
- moved R9 29.6 mm to (24.1, 49.5), turned to 180 degrees
- moved R8 29.0 mm to (40.6, 48.3)
- moved R6 23.2 mm to (36.8, 39.4)
- moved R3 21.6 mm to (38.1, 19.1), turned to 180 degrees
- moved R5 19.1 mm to (35.6, 30.5), turned to 0 degrees
- moved R10 14.8 mm to (30.5, 19.1)
- moved C7 12.7 mm to (22.9, 24.1), turned to 0 degrees
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Connections:
- removed net LDAC: B1.D9, U2.9
- removed net LDO+: C7.1, R14.2, R2.2, U1.12, U3.4
- removed net LDO-: C6.1, R3.2, U1.5, U3.11
- removed net N$24: R12.1, R13.2, U$7.1, U$8.1
- removed net N$25: R13.1, R19.1, U3.13
- removed net N$35: R20.2, U2.1
- removed net N$9: R6.1, R7.2, U$1.1, U$2.1
- removed net P_OUT1: J2.1, R18.2, U3.1
- removed net P_OUT2: J2.2, R17.2, U3.7
- removed net P_OUT3: J2.3, R16.2, U3.8
- removed net P_OUT4: J2.4, R19.2, U3.14
- removed net SCL: B1.SCL, U2.13
- removed net SDA: B1.SDA, U2.8
- removed net VOUTA: R6.2, U2.3
- removed net VOUTB: R8.2, U2.2
- removed net VOUTC: R10.2, U2.6
- removed net VOUTD: R12.2, U2.7
- removed net V_REF: R14.1, R15.2, U$9.1, U3.10, U3.12, U3.3, U3.5
- new net N$10: R3.1, R4.2, U3.2
- new net N$11: C7.1, QFM_SENSOR.4
- new net N$13: R5.1, U3.3
- new net N$14: R6.1, U2.6
- new net N$15: R7.1, U2.7
- new net N$17: R8.1, U2.10
- new net N$5: C2.2, U1.1
- new net VCC: J1.3, QFM_SENSOR.1, R10.3
- new net VDD3: C13.1, C14.1, U3.11
- net AGND: now also C1.2, C11.2, C12.2, C13.2, C14.2, C15.2, C16.2, C17.2, C18.2, C8.2, IC1.7, J1.1, QFM_SENSOR.3, R5.2, R6.2, R8.2, U1.4, U1.9, Y1.2; no longer C2.1, C3.2, C6.2, C7.2, J1.3, R1.1, R15.1, R4.1, R5.1, U$1.2, U$2.2, U$3.2, U$4.2, U$5.2, U$6.2, U$7.2, U$8.2, U$9.2, U1.14, U1.17, U2.14, U2.4
- net N$1: now also B1.D7, U1.8; no longer C5.1, U1.3
- net N$12: now also C7.2, R4.1, R7.2, U3.1; no longer R2.1, R4.2, U1.15
- net N$16: now also IC1.1, U2.1; no longer R18.1, R7.1, U3.2
- net N$18: now also R9.1, U2.11; no longer R8.1, R9.2, U$3.1, U$4.1
- net N$19: now also QFM_SENSOR.5, R9.2; no longer R17.1, R9.1, U3.6
- net N$2: now also U1.5, Y1.3; no longer R1.2, U1.2
- net N$21: now also IC1.2, U2.13; no longer R10.1, R11.2, U$5.1, U$6.1
- net N$22: now also B1.D8, IC1.3; no longer R11.1, R16.1, U3.9
- net N$3: now also B1.D6; no longer C1.1, U1.8
- net N$4: now also B1.D5, U1.6; no longer C1.2, U1.10, U1.9
- net N$6: now also C6.1, U1.10; no longer C3.1, U1.16
- net N$7: now also C3.2, U1.3; no longer C4.1, U1.6
- net N$8: now also C6.2, R10.2, R3.2; no longer R3.1, R5.2, U1.4
- net VDD: now also C1.1, C11.1, C12.1, C15.1, C16.1, C17.1, C18.1, C2.1, C3.1, C4.1, C5.1, C8.1, IC1.14, QFM_SENSOR.2, R10.1, U1.2, U2.3, U3.4, Y1.1, Y1.4; no longer C2.2, R20.1, U1.1, U1.11, U1.13, U2.10, U2.11, U2.15, U2.16, U2.5
Routing:
- net VDD: track 86.4 -> 198.7 mm, vias 4 -> 6
- net VCC: track 0.00 -> 100.5 mm, vias 0 -> 2
- net LDO-: track 71.1 -> 0.00 mm, vias 2 -> 0
- net VOUTC: track 44.1 -> 0.00 mm
- net LDAC: track 38.2 -> 0.00 mm, vias 2 -> 0
- net N$25: track 38.1 -> 0.00 mm, vias 2 -> 0
- net P_OUT2: track 37.9 -> 0.00 mm
- net VOUTD: track 36.5 -> 0.00 mm
- net LDO+: track 33.9 -> 0.00 mm, vias 2 -> 0
- net N$11: track 0.00 -> 30.7 mm
- net P_OUT1: track 30.6 -> 0.00 mm, vias 2 -> 0
- net V_REF: track 29.3 -> 0.00 mm, vias 2 -> 0
- net P_OUT4: track 29.1 -> 0.00 mm, vias 2 -> 0
- net N$15: track 0.00 -> 27.2 mm, vias 0 -> 2
- net N$22: track 22.3 -> 46.7 mm, vias 0 -> 2
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