File: electric/AFM_QFM_input.sch (EAGLE design)
At the start: 42 parts, among them U1 LTC3260EMSE#PBF, U2 AD5696RARUZ-RL7RU_16_ADI-M, U3 LM324KAD

Commit message: allboards
Parts:
- removed J2: (no value), SparkFun-Connectors:CONN_04LONGPADS
- removed R1: 220, SparkFun-Resistors:220OHM-0603-1/10W-1%
- removed R11, R12, R13: 5k, 52101-101-REV-A_v16:RC-MASTER-SMD_R_0603MP
- removed R14, R15, R20: 10k, 52101-101-REV-A_v16:RC-MASTER-SMD_R_0603MP
- removed R16, R17, R18, R19: 30k, 52101-101-REV-A_v16:RC-MASTER-SMD_R_0603MP
- removed R2: 100k, SparkFun-Resistors:100KOHM-0603-1/10W-1%
- removed U$1, U$3, U$5, U$7: 2.2uf, Nordic_nRF:CAPACITOR_0603_M
- removed U$2, U$4, U$6, U$8: 1uF, Nordic_nRF:CAPACITOR_0603_M
- removed U$9: 4.7uf, Nordic_nRF:CAPACITOR_0603_M
- added C11, C13, C15, C17: 0.1uF, SparkFun-Capacitors:0.1UF-0603-100V-10%
- added C12, C14, C16, C18, C8: 10uF, SparkFun-Capacitors:10UF-0805-10V-10%
- added IC1: 74HC86_SOIC, IC_Logic:74HC86_SOIC
- added QFM_SENSOR: (no value), SparkFun-Connectors:CONN_05PTH_LONGPADS
- added Y1: OSCILLATORSMD-5X3, SparkFun-Clocks:OSCILLATORSMD-5X3
- C1: value 1.0uF -> 0.1uF; device SparkFun-Capacitors:1.0UF-0805-25V-(+80/-20%) -> SparkFun-Capacitors:0.1UF-0603-100V-10%
- C2: value 10uF -> 10nF; device SparkFun-Capacitors:10UF-0805-25V-10% -> SparkFun-Capacitors:10NF-0603-50V-10%
- C3: value 10nF -> 0.1uF; device SparkFun-Capacitors:10NF-0603-50V-10% -> SparkFun-Capacitors:0.1UF-0603-100V-10%
- C4: value 10uF -> 0.1uF; device SparkFun-Capacitors:10UF-0805-25V-10% -> SparkFun-Capacitors:0.1UF-0603-100V-10%
- C5: value 10nF -> 10uF; device SparkFun-Capacitors:10NF-0603-50V-10% -> SparkFun-Capacitors:10UF-0805-10V-10%
- C6, C7: value 10uF -> 1.5nF; device SparkFun-Capacitors:10UF-0805-25V-10% -> resistor:C-EUC0603
- R10: value 5k -> 3224W-1-102E; device 52101-101-REV-A_v16:RC-MASTER-SMD_R_0603MP -> 3224W-1-102E:3224W-1-102E
- R3: value 100k -> (none); device SparkFun-Resistors:100KOHM-0603-1/10W-1% -> rcl:R-US_R0603
- R4, R5: value 300k -> (none); device SparkFun-Resistors:300KOHM-0603-1/10W-1% -> rcl:R-US_R0603
- R6, R7, R8, R9: value 5k -> (none); device 52101-101-REV-A_v16:RC-MASTER-SMD_R_0603MP -> rcl:R-US_R0603
- U1: value LTC3260EMSE#PBF -> AD9833BRM; device LTC3260EMSE_PBF (1):LTC3260EMSE#PBF -> AD9833BRM:AD9833BRM
- U2: value AD5696RARUZ-RL7RU_16_ADI-M -> LM339D; device AD5696:AD5696RARUZ-RL7RU_16_ADI-M -> LM339D:LM339D
Connections:
- removed net LDAC: B1.*D9, U2.!LDAC
- removed net LDO+: C7.1, R14.2, R2.2, U1.LDO+, U3.VCC+
- removed net LDO-: C6.1, R3.2, U1.LDO-, U3.VCC-
- removed net N$24: R12.1, R13.2, U$7.1, U$8.1
- removed net N$25: R13.1, R19.1, U3.NEG_4
- removed net N$35: R20.2, U2.VREF
- removed net N$9: R6.1, R7.2, U$1.1, U$2.1
- removed net P_OUT1: J2.1, R18.2, U3.OUT1
- removed net P_OUT2: J2.2, R17.2, U3.OUT2
- removed net P_OUT3: J2.3, R16.2, U3.OUT3
- removed net P_OUT4: J2.4, R19.2, U3.OUT4
- removed net SCL: B1.SCL, U2.SCL
- removed net SDA: B1.SDA, U2.SDA
- removed net VOUTA: R6.2, U2.VOUTA
- removed net VOUTB: R8.2, U2.VOUTB
- removed net VOUTC: R10.2, U2.VOUTC
- removed net VOUTD: R12.2, U2.VOUTD
- removed net V_REF: R14.1, R15.2, U$9.1, U3.POS_1, U3.POS_2, U3.POS_3, U3.POS_4
- new net N$10: R3.1, R4.2, U3.NEG_1
- new net N$11: C7.1, QFM_SENSOR.4
- new net N$13: R5.1, U3.POS_1
- new net N$14: R6.1, U2.1IN-
- new net N$15: R7.1, U2.1IN+
- new net N$17: R8.1, U2.4IN-
- new net N$5: C2.2, U1.COMP
- new net VCC: J1.3, QFM_SENSOR.1, R10.3
- new net VDD3: C13.1, C14.1, U3.VCC-
- net AGND: now also C1.2, C11.2, C12.2, C13.2, C14.2, C15.2, C16.2, C17.2, C18.2, C8.2, IC1.GND, J1.1, QFM_SENSOR.3, R5.2, R6.2, R8.2, U1.AGND, U1.DGND, Y1.GND; no longer C2.1, C3.2, C6.2, C7.2, J1.3, R1.1, R15.1, R4.1, R5.1, U$1.2, U$2.2, U$3.2, U$4.2, U$5.2, U$6.2, U$7.2, U$8.2, U$9.2, U1.EPAD, U1.MODE, U2.A0, U2.A1
- net N$1: now also B1.D7, U1.FSYNC; no longer C5.1, U1.BYP-
- net N$12: now also C7.2, R4.1, R7.2, U3.OUT1; no longer R2.1, R4.2, U1.ADJ+
- net N$16: now also IC1.1A, U2.1OUT; no longer R18.1, R7.1, U3.NEG_1
- net N$18: now also R9.1, U2.4IN+; no longer R8.1, R9.2, U$3.1, U$4.1
- net N$19: now also QFM_SENSOR.5, R9.2; no longer R17.1, R9.1, U3.NEG_2
- net N$2: now also U1.MCLK, Y1.OUT; no longer R1.2, U1.RT
- net N$21: now also IC1.1B, U2.OUT4; no longer R10.1, R11.2, U$5.1, U$6.1
- net N$22: now also B1.D8, IC1.1Y; no longer R11.1, R16.1, U3.NEG3
- net N$3: now also B1.*D6, U1.SCLK; no longer C1.1, U1.C-, U1.NC_2
- net N$4: now also B1.*D5, U1.SDATA; no longer C1.2, U1.C+, U1.NC
- net N$6: now also C6.1, U1.VOUT; no longer C3.1, U1.BYP+
- net N$7: now also C3.2, U1.CAP/2.5V; no longer C4.1, U1.VOUT
- net N$8: now also C6.2, R10.2, R3.2; no longer R3.1, R5.2, U1.ADJ-
- net VDD: now also C1.1, C11.1, C12.1, C15.1, C16.1, C17.1, C18.1, C2.1, C3.1, C4.1, C5.1, C8.1, IC1.VCC, QFM_SENSOR.2, R10.1, U1.VDD, U2.VCC, U3.VCC+, Y1.EN, Y1.VCC; no longer C2.2, R20.1, U1.EN+, U1.EN-, U1.VIN, U2.!RESET, U2.GAIN, U2.RSTSEL, U2.VDD, U2.VLOGIC
Other:
- moved on the sheet: B1, C1, C2, C3, C4, C5, C6, C7, R3, R4, R5, R6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
