File: electric/AFM_Power_board__ALL_SMD.brd (EAGLE design)
At the start: 68.2 x 57.1 mm, 18 parts, among them IC2 7815T, IC4 7805T, J2 694103303002

Commit message: newer electroincs
Parts:
- removed IC2: 7815T, adafruit:TO220H
- removed IC4: 7805T, adafruit:TO220H
- added C13: 1.0uF, SparkFun-Capacitors:0805
- added C14, C16, C18, C19: 10uF, SparkFun-Capacitors:0805
- added C15, C17: 10nF, SparkFun-Capacitors:0603
- added R3: 220, SparkFun-Resistors:0603
- added R4, R5: 100k, SparkFun-Resistors:0603
- added R6, R7: 300k, SparkFun-Resistors:0603
- added U2: LTC3260EMSE#PBF, LTC3260EMSE_PBF (1):MSOP-16_MSE
Connections:
- removed net N$2: D5.A, D6.C, J2.2, J2.3
- new net LDO+: C19.1, R4.2, U2.12
- new net LDO-: C18.1, R5.2, U2.5
- new net N$10: D6.A
- new net N$12: C17.1, U2.3
- new net N$13: C15.1, U2.16
- new net N$14: C16.1, U2.6
- new net N$15: R3.2, U2.2
- new net N$16: R5.1, R7.2, U2.4
- new net N$17: R4.1, R6.2, U2.15
- new net N$6: C13.1, U2.7, U2.8
- new net N$7: C13.2, U2.10, U2.9
- new net N$9: D5.A, D6.C
- new net S$1: J2.3
- new net S$3: C1.+, C2.1, C3.1
- new net S$4: C2.2, C3.2, L4.1
- new net S$6: J4.2
- new net V15+: U2.1, U2.11, U2.13
- net AGND: now also C14.1, C15.2, C16.2, C17.2, C18.2, C19.2, R3.1, R6.1, R7.1, U2.14, U2.17; no longer B1.GND@2, IC2.2, IC4.2
- net GROUND: no longer C2.2, C3.2, D2.A, D6.A, L4.1
- net N$1: no longer C6.1, C7.1, IC2.3, IC4.1
- net N$11: no longer C1.+, C2.1, C3.1, D5.C, L3.1
- net N$5: no longer IC2.1
- net V5_OUT: no longer C4.1, IC4.3, J4.2
Routing:
- net N$2: track 36.1 -> 0.00 mm
- net VMINUS5_OUT: track 46.3 -> 82.2 mm
- net N$11: track 52.4 -> 19.8 mm
- net N$1: track 93.6 -> 72.7 mm
- net N$9: track 0.00 -> 19.3 mm
- net S$4: track 0.00 -> 17.6 mm
- net V5_OUT: track 35.7 -> 20.1 mm
- net S$6: track 0.00 -> 14.4 mm
- net S$3: track 0.00 -> 13.2 mm
- net GROUND: track 28.5 -> 23.8 mm, vias 0 -> 2
- net S$5: track 0.00 -> 3.07 mm
- net N$10: track 0.00 -> 2.69 mm
- net S$1: track 0.00 -> 0.50 mm
