File: electric/AFM_Power_board__ALL_SMD.sch (EAGLE design)
At the start: 18 parts, among them IC2 7815T, IC4 7805T, J2 694103303002

Commit message: newer electroincs
Parts:
- removed IC2: 7815T, adafruit:7815T
- removed IC4: 7805T, adafruit:7805T
- added IC1: LM7805_SOT223, IC_Power-Management:LM7805_SOT223
- added IC3: 7815DT, adafruit:7815DT
Connections:
- removed net N$1 (its old number): C6.1, C7.1, IC2.VO, IC4.VI, J4.4
- new net V15+: C6.1, C7.1, IC1.VI, IC3.VO, J4.4
- net AGND: now also IC1.GND, IC3.GND; no longer IC2.GND, IC4.GND
- net N$5: now also IC3.VI; no longer IC2.VI
- net V5_OUT: now also IC1.VO; no longer IC4.VO
Changed lines of the file:
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@@
 <part name="D3" library="diode" library_urn="urn:adsk.eagle:library:210" deviceset="DIODE-" device="SOD123" package3d_urn="urn:adsk.eagle:package:43420/1" value="1n4004"/>
 <part name="J4" library="SparkFun-Connectors" library_urn="urn:adsk.eagle:library:513" deviceset="CONN_04" device="LONGPADS" package3d_urn="urn:adsk.eagle:package:38098/2"/>
-<part name="IC2" library="adafruit" library_urn="urn:adsk.eagle:library:420" deviceset="78*" device="T" package3d_urn="urn:adsk.eagle:package:6240670/1" technology="15"/>
 <part name="C6" library="BeagleBone_Black_Wireless" library_urn="urn:adsk.eagle:library:6644236" deviceset="C-US" device="050-024X044" package3d_urn="urn:adsk.eagle:package:8118541/1" value="10uF"/>
 <part name="C7" library="BeagleBone_Black_Wireless" library_urn="urn:adsk.eagle:library:6644236" deviceset="C-US" device="050-024X044" package3d_urn="urn:adsk.eagle:package:8118541/1" value="1uF"/>
-<part name="IC4" library="adafruit" library_urn="urn:adsk.eagle:library:420" deviceset="78*" device="T" package3d_urn="urn:adsk.eagle:package:6240670/1" technology="05"/>
+<part name="IC1" library="IC_Power-Management" library_urn="urn:adsk.eagle:library:16378392" deviceset="LM7805" device="_SOT223" package3d_urn="urn:adsk.eagle:package:16494942/2"/>
+<part name="IC3" library="adafruit" library_urn="urn:adsk.eagle:library:420" deviceset="78*" device="DT" package3d_urn="urn:adsk.eagle:package:6240672/1" technology="15"/>
 </parts>
 <sheets>
@@
 <attribute name="NAME" x="107.188" y="124.46" size="1.778" layer="95" font="vector" rot="R270"/>
 </instance>
-<instance part="IC2" gate="A1" x="22.86" y="109.22" smashed="yes">
-<attribute name="NAME" x="15.24" y="114.935" size="1.778" layer="95"/>
-<attribute name="VALUE" x="15.24" y="112.395" size="1.778" layer="96"/>
-</instance>
 <instance part="C6" gate="G$1" x="38.1" y="96.52" smashed="yes">
 <attribute name="NAME" x="39.116" y="97.155" size="1.778" layer="95"/>
@@
 <attribute name="VALUE" x="49.276" y="92.329" size="1.778" layer="96"/>
 </instance>
-<instance part="IC4" gate="A1" x="68.58" y="109.22" smashed="yes">
-<attribute name="NAME" x="60.96" y="114.935" size="1.778" layer="95"/>
-<attribute name="VALUE" x="60.96" y="112.395" size="1.778" layer="96"/>
+<instance part="IC1" gate="G$1" x="68.58" y="109.22" smashed="yes">
+<attribute name="NAME" x="68.58" y="113.22" size="1.778" layer="95" align="center"/>
+<attribute name="VALUE" x="71.12" y="102.22" size="1.778" layer="96" align="center-left"/>
+</instance>
+<instance part="IC3" gate="A1" x="22.86" y="109.22" smashed="yes">
+<attribute name="NAME" x="15.24" y="114.935" size="1.778" layer="95"/>
+<attribute name="VALUE" x="15.24" y="112.395" size="1.778" layer="96"/>
 </instance>
 </instances>
@@
 <junction x="68.58" y="86.36"/>
 <pinref part="J4" gate="J1" pin="1"/>
-<pinref part="IC2" gate="A1" pin="GND"/>
 <wire x1="22.86" y1="101.6" x2="22.86" y2="86.36" width="0.1524" layer="91"/>
 <junction x="22.86" y="86.36"/>
@@
 <wire x1="48.26" y1="91.44" x2="48.26" y2="86.36" width="0.1524" layer="91"/>
 <junction x="48.26" y="86.36"/>
-<pinref part="IC4" gate="A1" pin="GND"/>
+<pinref part="IC1" gate="G$1" pin="GND"/>
+<pinref part="IC3" gate="A1" pin="GND"/>
 </segment>
 </net>
@@
 <junction x="91.44" y="93.98"/>
 <pinref part="J4" gate="J1" pin="2"/>
-<pinref part="IC4" gate="A1" pin="VO"/>
 <wire x1="78.74" y1="109.22" x2="91.44" y2="109.22" width="0.1524" layer="91"/>
+<pinref part="IC1" gate="G$1" pin="VO"/>
 </segment>
 </net>
@@
 <wire x1="-50.8" y1="81.28" x2="-48.26" y2="81.28" width="0.1524" layer="91"/>
 <junction x="-50.8" y="81.28"/>
-<wire x1="-48.26" y1="81.28" x2="-48.26" y2="71.12" width="0.1524" layer="91"/>
-<wire x1="-48.26" y1="71.12" x2="-27.94" y2="71.12" width="0.1524" layer="91"/>
+<wire x1="-48.26" y1="81.28" x2="-48.26" y2="63.5" width="0.1524" layer="91"/>
 <pinref part="D2" gate="G$1" pin="A"/>
 <pinref part="D6" gate="G$1" pin="A"/>
-<wire x1="-27.94" y1="71.12" x2="-27.94" y2="86.36" width="0.1524" layer="91"/>
+<wire x1="-48.26" y1="63.5" x2="-35.56" y2="63.5" width="0.1524" layer="91"/>
+<wire x1="-35.56" y1="63.5" x2="-35.56" y2="86.36" width="0.1524" layer="91"/>
+<junction x="-35.56" y="86.36"/>
 </segment>
 </net>
@@
 <wire x1="149.86" y1="104.14" x2="149.86" y2="63.5" width="0.1524" layer="91"/>
 <wire x1="149.86" y1="63.5" x2="96.52" y2="63.5" width="0.1524" layer="91"/>
-<wire x1="96.52" y1="63.5" x2="96.52" y2="71.12" width="0.1524" layer="91"/>
 <pinref part="J4" gate="J1" pin="3"/>
 </segment>
@@
 </segment>
 </net>
-<net name="N$1" class="0">
-<segment>
-<pinref part="IC2" gate="A1" pin="VO"/>
+<net name="N$3" class="0">
+<segment>
+<wire x1="5.08" y1="93.98" x2="5.08" y2="91.44" width="0.1524" layer="91"/>
+</segment>
+</net>
+<net name="N$5" class="0">
+<segment>
+<wire x1="12.7" y1="109.22" x2="7.62" y2="109.22" width="0.1524" layer="91"/>
+<wire x1="7.62" y1="109.22" x2="7.62" y2="93.98" width="0.1524" layer="91"/>
+<pinref part="L3" gate="G$1" pin="2"/>
+<wire x1="7.62" y1="93.98" x2="0" y2="93.98" width="0.1524" layer="91"/>
+<pinref part="IC3" gate="A1" pin="VI"/>
+</segment>
+</net>
+<net name="V15+" class="0">
+<segment>
 <wire x1="33.02" y1="109.22" x2="38.1" y2="109.22" width="0.1524" layer="91"/>
 <pinref part="C6" gate="G$1" pin="1"/>
@@
 <wire x1="88.9" y1="116.84" x2="38.1" y2="116.84" width="0.1524" layer="91"/>
 <wire x1="38.1" y1="116.84" x2="38.1" y2="109.22" width="0.1524" layer="91"/>
-<pinref part="IC4" gate="A1" pin="VI"/>
-</segment>
-</net>
-<net name="N$3" class="0">
-<segment>
-<wire x1="5.08" y1="93.98" x2="5.08" y2="91.44" width="0.1524" layer="91"/>
-</segment>
-</net>
-<net name="N$5" class="0">
-<segment>
-<pinref part="IC2" gate="A1" pin="VI"/>
-<wire x1="12.7" y1="109.22" x2="7.62" y2="109.22" width="0.1524" layer="91"/>
-<wire x1="7.62" y1="109.22" x2="7.62" y2="93.98" width="0.1524" layer="91"/>
-<pinref part="L3" gate="G$1" pin="2"/>
-<wire x1="7.62" y1="93.98" x2="0" y2="93.98" width="0.1524" layer="91"/>
-</segment>
-</net>
-<net name="N$2" class="0">
+<wire x1="104.14" y1="111.76" x2="215.9" y2="111.76" width="0.1524" layer="91"/>
+<junction x="104.14" y="111.76"/>
+<pinref part="IC1" gate="G$1" pin="VI"/>
+<pinref part="IC3" gate="A1" pin="VO"/>
+</segment>
+</net>
+<net name="N$1" class="0">
 <segment>
 <pinref part="J2" gate="G$1" pin="2"/>
