File: electric/AFM_Power_board__NEW.brd (EAGLE design)
At the start: 68.2 x 57.1 mm, 18 parts, among them IC2 7815T, IC4 7805T, J2 694103303002

Commit message: newer electroincs
Parts:
- added C10, C12: 1uF, BeagleBone_Black_Wireless:C050-024X044
- added C11, C9: 10uF, BeagleBone_Black_Wireless:C050-024X044
- added C8: 220uF, BeagleBone_Blue_R3:E5-8,5
- added IC1, IC3: LM4041CILP, texas:LP_O-PBCY-W3
- added J3: 694103303002, DC Power Jacks:694103303002
- added L1: 60Ohm@100 MHz, Wurth_EMC Components_WE-CBF:WE-CBF_0603_W2.2
- added R1, R2: (no value), BeagleBone_Black_Wireless:0204/5
- added U1: LM7905CT/NOPB, LM7905CT_NOPB:TO254P1016X4575X1955-3
Connections:
- new net N$10: C10.2, C8.-, C9.2, D2.A, D6.A, L1.1
- new net N$4: IC1.2, R1.2
- new net N$8: IC3.3, R2.2
- new net N$9: D5.A, D6.C, J3.1
- net AGND: now also C11.1, C12.1, IC1.3, IC3.2, U1.1
- net GROUND: now also C10.1, C8.+, C9.1, J2.2, J2.3, J3.2, J3.3; no longer D2.A, D6.A
- net N$2: now also L1.2, U1.2; no longer D5.A, D6.C, J2.2, J2.3
- net V5_OUT: now also R1.1
- net VMINUS5_OUT: now also C11.2, C12.2, R2.1, U1.3
Routing:
- net GROUND: track 28.5 -> 83.5 mm, vias 0 -> 2
- net VMINUS5_OUT: track 46.3 -> 100.5 mm
- net N$10: track 0.00 -> 38.0 mm
- net N$2: track 36.1 -> 7.47 mm
- net N$9: track 0.00 -> 20.5 mm
- net V5_OUT: track 35.7 -> 48.4 mm
- net N$4: track 0.00 -> 11.2 mm
- net N$8: track 0.00 -> 5.61 mm
