File: electric/AFM_QFM_input__smd_xor.brd (EAGLE design)
At the start: 64.4 x 55.9 mm, 31 parts, among them U1 AD9833BRM, U2 LM339D, U3 LM324KAD, U4 SN74LVC1G86DCKRG4, Y1 OSCILLATORSMD-5X3

Commit message: newer electroincs
Parts:
- removed J2: (no value), SparkFun-Connectors:1X04_LONGPADS
- added J1: (no value), SparkFun-Connectors:1X03_LONGPADS
- R3: value 7.2k -> (none)
- R4: value 100k -> (none)
- R5: value 1k -> (none)
- R6: value 5,6k -> (none)
- R7, R8, R9: value 5.6k -> (none)
- moved U4 1.27 mm to (24.1, 44.5)
Connections:
- net AGND: now also J1.1; no longer J2.1
- net VCC: now also J1.3; no longer J2.3
- net VDD3: now also J1.2; no longer J2.2
Routing:
- net AGND: track 43.9 -> 38.3 mm, vias 2 -> 1
- net N$7: track 4.35 -> 8.62 mm
- net N$22: track 69.1 -> 71.2 mm
- net VDD3: track 157.3 -> 156.1 mm
- net N$1: track 15.4 -> 16.3 mm
- net N$2: track 4.39 -> 5.28 mm, vias 1 -> 0
- net VCC: track 154.1 -> 153.2 mm, vias 3 -> 4
- net N$3: track 13.4 -> 14.0 mm
- net N$21: track 13.5 -> 14.0 mm, vias 1 -> 0
- net N$16: track 10.0 -> 9.48 mm, vias 1 -> 0
- net N$11: vias 1 -> 0
