File: electric/AFM_QFM_input__smd_xor.sch (EAGLE design)
At the start: 31 parts, among them U1 AD9833BRM, U2 LM339D, U3 LM324KAD, U4 SN74LVC1G86DCKRG4, Y1 OSCILLATORSMD-5X3

Commit message: newer electroincs
Parts:
- removed J2: (no value), SparkFun-Connectors:CONN_04LONGPADS
- added J1: (no value), SparkFun-Connectors:CONN_03LONGPADS
Connections:
- net AGND: now also J1.1; no longer J2.2
- net VCC: now also J1.3; no longer J2.4
- net VDD3: now also J1.2; no longer J2.3
Changed lines of the file:
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@@
 <parts>
 <part name="B1" library="SparkFun-Boards" library_urn="urn:adsk.eagle:library:509" deviceset="ARDUINO_UNO_R3_SHIELD" device="BASIC" package3d_urn="urn:adsk.eagle:package:41384914/1"/>
+<part name="J1" library="SparkFun-Connectors" library_urn="urn:adsk.eagle:library:513" deviceset="CONN_03" device="LONGPADS" package3d_urn="urn:adsk.eagle:package:38068/2"/>
 <part name="SUPPLY2" library="Power_Symbols" library_urn="urn:adsk.eagle:library:16502351" deviceset="AGND" device="" value="AGND"/>
 <part name="U3" library="LM324KAD" deviceset="LM324KAD" device=""/>
@@
 <part name="SUPPLY5" library="Power_Symbols" library_urn="urn:adsk.eagle:library:16502351" deviceset="AGND" device="" value="AGND"/>
 <part name="U4" library="SN74LVC1G86DCKRG4" deviceset="SN74LVC1G86DCKRG4" device=""/>
-<part name="J2" library="SparkFun-Connectors" library_urn="urn:adsk.eagle:library:513" deviceset="CONN_04" device="LONGPADS" package3d_urn="urn:adsk.eagle:package:38098/2"/>
 </parts>
 <sheets>
@@
 <attribute name="VALUE" x="199.39" y="-53.594" size="1.778" layer="96" font="vector" align="top-left"/>
 </instance>
+<instance part="J1" gate="J1" x="99.06" y="116.84" smashed="yes" rot="R270">
+<attribute name="VALUE" x="91.694" y="119.38" size="1.778" layer="96" font="vector" rot="R270"/>
+<attribute name="NAME" x="104.648" y="119.38" size="1.778" layer="95" font="vector" rot="R270"/>
+</instance>
 <instance part="SUPPLY2" gate="G$1" x="96.52" y="91.44" smashed="yes">
 <attribute name="VALUE" x="96.393" y="87.757" size="1.778" layer="96" align="bottom-center"/>
@@
 <attribute name="NAME" x="325.12" y="82.28" size="2.0828" layer="95" ratio="10" rot="SR0"/>
 <attribute name="VALUE" x="325.12" y="56.96" size="2.0828" layer="96" ratio="10" rot="SR0"/>
-</instance>
-<instance part="J2" gate="J1" x="96.52" y="114.3" smashed="yes" rot="R270">
-<attribute name="VALUE" x="89.154" y="119.38" size="1.778" layer="96" font="vector" rot="R270"/>
-<attribute name="NAME" x="104.648" y="119.38" size="1.778" layer="95" font="vector" rot="R270"/>
 </instance>
 </instances>
@@
 <wire x1="96.52" y1="93.98" x2="86.36" y2="93.98" width="0.1524" layer="91"/>
 <pinref part="SUPPLY2" gate="G$1" pin="AGND"/>
+<pinref part="J1" gate="J1" pin="1"/>
 <wire x1="96.52" y1="109.22" x2="96.52" y2="93.98" width="0.1524" layer="91"/>
 <wire x1="86.36" y1="93.98" x2="86.36" y2="58.42" width="0.1524" layer="91"/>
@@
 <pinref part="C8" gate="G$1" pin="2"/>
 <wire x1="45.72" y1="48.26" x2="45.72" y2="50.8" width="0.1524" layer="91"/>
-<pinref part="J2" gate="J1" pin="2"/>
 </segment>
 <segment>
@@
 <net name="VCC" class="0">
 <segment>
+<pinref part="J1" gate="J1" pin="3"/>
 <wire x1="101.6" y1="109.22" x2="101.6" y2="106.68" width="0.1524" layer="91"/>
 <wire x1="101.6" y1="106.68" x2="205.74" y2="106.68" width="0.1524" layer="91"/>
@@
 <wire x1="223.52" y1="106.68" x2="205.74" y2="106.68" width="0.1524" layer="91"/>
 <junction x="205.74" y="106.68"/>
-<pinref part="J2" gate="J1" pin="4"/>
 </segment>
 </net>
@@
 <net name="VDD3" class="0">
 <segment>
+<pinref part="J1" gate="J1" pin="2"/>
 <wire x1="99.06" y1="106.68" x2="99.06" y2="109.22" width="0.1524" layer="91"/>
 <label x="91.44" y="106.68" size="1.778" layer="95"/>
@@
 <pinref part="U4" gate="A" pin="VCC"/>
 <wire x1="368.3" y1="78.74" x2="355.6" y2="78.74" width="0.1524" layer="91"/>
-<pinref part="J2" gate="J1" pin="3"/>
-</segment>
-</net>
+</segment>
+</net>
