File: electric/AFM_QFM_sensor_OPA656NB.sch (EAGLE design)
At the start: 22 parts, among them J4 USBR-A-S-S-O-TH, U2 AD8676ARMZ, U3 AD8675ARMZ-REEL, U4 OPA656U

Commit message: newer electroincs
Parts:
- removed U4: OPA656U, OPA656U:OPA656U
- added U1: OPA656NB/250, OPA656NB_250:OPA656NB/250
Connections:
- net AGND: now also U1.POS_IN; no longer U4.POS
- net N$3: now also U1.NEG_IN; no longer U4.NEG
- net OPA_OUT: now also U1.OUT; no longer U4.OUTPUT
- net V+: now also U1.+VS; no longer U4.+VS
- net V-: now also U1.-VS; no longer U4.-VS
Changed lines of the file:
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@@
 <part name="C11" library="SparkFun-Capacitors" library_urn="urn:adsk.eagle:library:510" deviceset="10UF" device="-0805-10V-10%" package3d_urn="urn:adsk.eagle:package:41385092/1" value="10uF"/>
 <part name="J4" library="USBR-A-S-S-O-TH" deviceset="USBR-A-S-S-O-TH" device=""/>
-<part name="U4" library="OPA656U" deviceset="OPA656U" device=""/>
+<part name="U1" library="OPA656NB_250" deviceset="OPA656NB/250" device=""/>
 </parts>
 <sheets>
@@
 <attribute name="VALUE" x="12.7" y="135.89" size="1.778" layer="96" rot="R180" align="top-left"/>
 </instance>
-<instance part="U4" gate="A" x="66.04" y="81.28" smashed="yes">
+<instance part="U1" gate="A" x="66.04" y="81.28" smashed="yes">
 <attribute name="NAME" x="53.34" y="92.44" size="2.0828" layer="95" ratio="10" rot="SR0"/>
 <attribute name="VALUE" x="53.34" y="67.12" size="2.0828" layer="96" ratio="10" rot="SR0"/>
@@
 <junction x="104.14" y="81.28"/>
 <label x="149.86" y="71.12" size="1.778" layer="95"/>
-<pinref part="U4" gate="A" pin="-VS"/>
+<pinref part="U1" gate="A" pin="-VS"/>
 </segment>
 </net>
@@
 <junction x="109.22" y="91.44"/>
 <junction x="116.84" y="91.44"/>
-<pinref part="U4" gate="A" pin="POS"/>
+<pinref part="U1" gate="A" pin="POS_IN"/>
 </segment>
 <segment>
@@
 <pinref part="J4" gate="G$1" pin="D-"/>
 <wire x1="17.78" y1="121.92" x2="22.86" y2="121.92" width="0.1524" layer="91"/>
-<pinref part="U4" gate="A" pin="NEG"/>
+<pinref part="U1" gate="A" pin="NEG_IN"/>
 </segment>
 </net>
@@
 <junction x="104.14" y="50.8"/>
 <label x="86.36" y="78.74" size="1.778" layer="95"/>
-<pinref part="U4" gate="A" pin="OUTPUT"/>
+<pinref part="U1" gate="A" pin="OUT"/>
 </segment>
 </net>
@@
 <wire x1="129.54" y1="88.9" x2="139.7" y2="88.9" width="0.1524" layer="91"/>
 <wire x1="139.7" y1="88.9" x2="139.7" y2="73.66" width="0.1524" layer="91"/>
-<pinref part="U4" gate="A" pin="+VS"/>
-</segment>
-</net>
+<pinref part="U1" gate="A" pin="+VS"/>
+</segment>
+</net>
